File: hardware/motherboard.sch (EAGLE design)
At the start: 46 parts, among them IC1 7805T, Q1 16MHz, U1 ATMEGA328P-PU, U2 L293NE

Commit message: Added partlists for boards.
Parts:
- C1: device resistor:C-EUC1206K -> resistor:C-EUC0805K
Changed lines of the file:
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@@
 <?xml version="1.0" encoding="utf-8"?>
 <!DOCTYPE eagle SYSTEM "eagle.dtd">
-<eagle version="7.5.0">
+<eagle version="7.6.0">
 <drawing>
 <settings>
@@
 <setting verticaltext="up"/>
 </settings>
-<grid distance="0.1" unitdist="inch" unit="inch" style="lines" multiple="1" display="no" altdistance="0.01" altunitdist="inch" altunit="inch"/>
+<grid distance="0.1" unitdist="inch" unit="inch" style="lines" multiple="1" display="yes" altdistance="0.05" altunitdist="inch" altunit="inch"/>
 <layers>
 <layer number="1" name="Top" color="4" fill="1" visible="no" active="no"/>
@@
 <part name="IC1" library="linear" deviceset="78*" device="T" technology="05"/>
 <part name="P+2" library="supply1" deviceset="VCC" device=""/>
-<part name="C1" library="resistor" deviceset="C-EU" device="C1206K" value="330n"/>
+<part name="C1" library="resistor" deviceset="C-EU" device="C0805K" value="330n"/>
 <part name="C2" library="resistor" deviceset="CPOL-EU" device="E2.5-5" value="100u"/>
 <part name="P+3" library="supply1" deviceset="VCC" device=""/>

Commit message: Beautified sensorboard and motherboard schematics. Fixed motherboard angle error.
Other:
- moved on the sheet: C1, C2, C3, C4, C5, C6, C7, C8, C9, D1, D10, D2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
